File: badge24.kicad_pcb (KiCad board)
At the start: 2 copper layers, 111.2 x 110.3 mm, 23 parts, among them J1 SAO CONNECTOR, J2 SAO CONNECTOR, J3 SAO CONNECTOR, J4 SAO CONNECTOR, J5 SAO CONNECTOR, J6 SAO CONNECTOR, J7 Conn_01x09, J99 VEXT, M1 SC0918, SW11 SW_Push, SW22 SW_Push, SW33 SW_Push, T1 DMG2305

Commit message: clean up for writeup
Parts:
- BT1, BT2: footprint .stumbler:BatteryHolder_Keystone_2460_1xAA_SAO -> .badge24:BatteryHolder_Keystone_2460_1xAA_SAO
- J1, J2, J3, J4, J5, J6: footprint .stumbler:SAO_PIN_HEADER_2x03 -> .badge24:SAO_PIN_HEADER_2x03
- J7: footprint .stumbler:IO_SAO_1x09_SMD_EXTERNAL -> .badge24:IO_SAO_1x09_SMD_EXTERNAL
- J99: footprint .stumbler:SAO_PinHeader_1x02_P2.54mm_SMD -> .badge24:SAO_PinHeader_1x02_P2.54mm_SMD
- JP1: footprint .stumbler:SolderJumper_Open_Rounded_SAO -> .badge24:SolderJumper_Open_Rounded_SAO
- LD1: footprint LED_SMD:LED_0805_2012Metric -> .badge24:LED_0805_2012Metric
- M1: footprint .stumbler:RPi_Pico_SMD_SAO -> .badge24:RPi_Pico_SMD_SAO
- R1, R2, R3, R4, R5: footprint .stumbler:R_0603_1608Metric_SAO -> .badge24:R_0603_1608Metric_SAO
- S1: footprint Button_Switch_THT:SW_Slide-03_Wuerth-WS-SLTV_10x2.5x6.4_P2.54mm -> .badge24:SW_Slide-03_Wuerth-WS-SLTV_10x2.5x6.4_P2.54mm; moved to B.Cu
- SW11, SW22, SW33: footprint .stumbler:SW_SPST_PTS645_SAO -> .badge24:SW_SPST_PTS645_SAO
- T1: footprint .stumbler:SOT-23_SAO -> .badge24:SOT-23_SAO
- moved J1 15.0 mm to (109.3, 58.6)
- moved J6 15.0 mm to (195.7, 58.9)
- moved BT1 15.0 mm to (129.1, 78.3)
- moved BT2 15.0 mm to (171.5, 78.4)
- moved J2 15.0 mm to (96.3, 102.4)
- moved J3 15.0 mm to (122.1, 138.7)
- moved J4 15.0 mm to (174.3, 139.6)
- moved J5 15.0 mm to (200.6, 104.2)
- moved J7 15.0 mm to (118.3, 87.8)
- moved J99 15.0 mm to (181.7, 68.9)
- moved JP1 15.0 mm to (184.6, 97.6)
- moved LD1 15.0 mm to (149.9, 115.3)
- moved M1 15.0 mm to (151.2, 104.7)
- moved R1 15.0 mm to (184.6, 89.6)
- moved R2 15.0 mm to (184.6, 93.4)
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Other:
- board text removed: "REDRAWN BY THE STUMBLER"
